File: usb_to_gpib.sch (KiCad schematic (older format))
At the start: 34 parts, among them P1 CONN_12X2, P2 CONN_6, P3 CONN_1, P4 CONN_1, SW1 SW_PUSH, U1 PIC18F4520, U2 SN75160B, U3 SN75162B, U4 FT230X, X1 CRYSTAL

Commit message: Some modifications:  * removed exotic dual resistors  * added usbpicprog compatible isp header  * smaller board  * usb mini connector
Parts:
- removed C13: 4.7nF, ~, symbol C
- removed CONN1: Conn1, symbol CONN
- removed L1: INDUCTOR, symbol INDUCTOR
- removed P2: CONN_6, symbol CONN_6
- removed P3, P4: CONN_1, symbol CONN_1
- removed RP1: 27ohm, ~, symbol R_PACK2
- removed RP2, RP3: 270ohm, ~, symbol R_PACK2
- removed SW1: SW_PUSH, symbol SW_PUSH
- added L1: INDUCTOR_SMALL, Resistors_SMD:R_0603, symbol INDUCTOR_SMALL
- added P2: CONN_01X05, Pin_Headers:Pin_Header_Straight_1x05, symbol CONN_01X05
- added P5: USB_OTG, Connect:USB_Mini-B, symbol USB_OTG
- added R3, R4, R5: 270 ohm, Resistors_SMD:R_0603, symbol R
- added R6, R7: 27 ohm, Resistors_SMD:R_0603, symbol R
- C1, C11, C2, C3, C4, C7, C8: footprint (none) -> Capacitors_SMD:C_0603; symbol C -> C-RESCUE-usb_to_gpib
- C10, C12, C5, C9: footprint ~ -> Capacitors_SMD:C_0603; symbol C -> C-RESCUE-usb_to_gpib
- C6: footprint (none) -> Capacitors_SMD:C_1210; symbol CP1 -> CP1-RESCUE-usb_to_gpib
- D1, D2, D3, D4: footprint (none) -> LEDs:LED_0805; symbol LED -> LED-RESCUE-usb_to_gpib
- P1: footprint (none) -> gpib_conn_male:gpib_conn_male
- R1: footprint (none) -> Resistors_SMD:R_0603; symbol R -> R-RESCUE-usb_to_gpib
- R2: value 1M -> 270 ohm; footprint ~ -> Resistors_SMD:R_0603
- X1: footprint (none) -> Crystals:ABM3
Connections:
- net labels added: USB_D_N, USB_D_P, mUSB_N, mUSB_P
- net labels removed: USB_D+, USB_D-
- wire segments 228 -> 183
- no-connect marks 14 -> 13
Other:
- moved on the sheet: P1, R1
